File: kicad/control-pilot.sch (KiCad schematic (older format))
At the start: 42 parts, among them J6 Screw_Terminal_01x03, Q1 AO3400, Q2 AO3401, Q3 AO3400, Q4 AO3401, SW3 SS-12D00G3, SW4 SS-12D00G3, U1 LM224

Commit message: ...
Parts:
- removed J6: Screw_Terminal_01x03, Project:screw-terminal-230v-16a-5mm-3pin, symbol Connector:Screw_Terminal_01x03
- added C6: 2.2n, Capacitors_THT:C_Disc_D3.8mm_W2.6mm_P2.50mm, symbol Device:C_Small
- added C7: 220n, Project:c-1206-hand-soldering, symbol Device:C_Small
- added C8: 1u, Project:c-1206-hand-soldering, symbol Device:C_Small
- added C9: 1n, Project:c-1206-hand-soldering, symbol Device:C_Small
- added D13: 1N4007, Project:sma_hand-soldering, symbol Device:D_Small
- added J6: Screw_Terminal_01x04, Project:screw-terminal-230v-16a-5mm-4pin, symbol Connector:Screw_Terminal_01x04
- added JP3: Jumper_NO_Small, Project:idc-header-1x02-p2.54mm-vertical, symbol Device:Jumper_NO_Small
- added R55: 820K, Project:r-1206-hand-soldering, symbol rpi-ev-plc-adapter-rescue:R-ev-charger-met16-rescue
- added R56: 100R, Project:r-0805-hand-soldering, symbol rpi-ev-plc-adapter-rescue:R-ev-charger-met16-rescue
- added R57: 39K, Project:r-0805-hand-soldering, symbol rpi-ev-plc-adapter-rescue:R-ev-charger-met16-rescue
- added U2: PC817C, Project:sop-4-pc817, symbol project:PC817C
Connections:
- net labels added: L, ZERODET
- net labels removed: CP-PWM
- wire segments 151 -> 186
