File: kicad/control-pilot.sch (KiCad schematic (older format))
At the start: 52 parts, among them J6 Screw_Terminal_01x04, Q1 AO3400, Q2 AO3401, Q3 AO3400, Q4 AO3401, SW3 SS-12D00G3, SW4 SS-12D00G3, U1 LM224, U2 PC817C

Commit message: pcb fix for modem with 1.27mm connector finished
Parts:
- C6: footprint Capacitors_THT:C_Disc_D3.8mm_W2.6mm_P2.50mm -> Project:c-1206-hand-soldering
Changed lines of the file:
@@
 F 0 "C6" H 7792 1841 50  0000 L CNN
 F 1 "2.2n" H 7792 1750 50  0000 L CNN
-F 2 "Capacitors_THT:C_Disc_D3.8mm_W2.6mm_P2.50mm" H 7700 1750 50  0001 C CNN
+F 2 "Project:c-1206-hand-soldering" H 7700 1750 50  0001 C CNN
 F 3 "~" H 7700 1750 50  0001 C CNN
 F 4 "1000V" H 7792 1659 50  0000 L CNN "type"

Commit message: schematic/pcb V1.0 finished
Parts:
- R10, R11, R12, R13, R14, R15, R16, R17, R18, R19, R20, R21, R22, R23, R24, R25, R26, R27, R28, R29, R30, R31, R32, R33, R34, R35, R56, R57: footprint Project:r-0805-hand-soldering -> Project:r-1206-hand-soldering
Changed lines of the file:
@@
 F 0 "R15" H 4350 3500 50  0000 C CNN
 F 1 "100k" H 4350 3400 50  0000 C CNN
-F 2 "Project:r-0805-hand-soldering" V 4430 3450 50  0001 C CNN
+F 2 "Project:r-1206-hand-soldering" V 4430 3450 50  0001 C CNN
 F 3 "" H 4500 3450 50  0001 C CNN
 	1    4500 3450
@@
 F 0 "R16" H 4350 4150 50  0000 C CNN
 F 1 "22k" H 4350 4050 50  0000 C CNN
-F 2 "Project:r-0805-hand-soldering" V 4430 4050 50  0001 C CNN
+F 2 "Project:r-1206-hand-soldering" V 4430 4050 50  0001 C CNN
 F 3 "" H 4500 4050 50  0001 C CNN
 	1    4500 4050
@@
 F 0 "R19" H 6425 4125 50  0000 C CNN
 F 1 "1G" H 6400 4025 50  0000 C CNN
-F 2 "Project:r-0805-hand-soldering" V 6230 4050 50  0001 C CNN
+F 2 "Project:r-1206-hand-soldering" V 6230 4050 50  0001 C CNN
 F 3 "" H 6300 4050 50  0001 C CNN
 	1    6300 4050
@@
 F 0 "R17" H 5650 1350 50  0000 C CNN
 F 1 "2.74k" H 5650 1250 50  0000 C CNN
-F 2 "Project:r-0805-hand-soldering" V 5730 1300 50  0001 C CNN
+F 2 "Project:r-1206-hand-soldering" V 5730 1300 50  0001 C CNN
 F 3 "" H 5800 1300 50  0001 C CNN
 	1    5800 1300
@@
 F 0 "R18" H 6150 1350 50  0000 C CNN
 F 1 "1.3k" H 6150 1250 50  0000 C CNN
-F 2 "Project:r-0805-hand-soldering" V 5930 1300 50  0001 C CNN
+F 2 "Project:r-1206-hand-soldering" V 5930 1300 50  0001 C CNN
 F 3 "" H 6000 1300 50  0001 C CNN
 	1    6000 1300
@@
 F 0 "R20" H 3425 2300 50  0000 C CNN
 F 1 "1k" H 3400 2225 50  0000 C CNN
-F 2 "Project:r-0805-hand-soldering" V 3230 2250 50  0001 C CNN
+F 2 "Project:r-1206-hand-soldering" V 3230 2250 50  0001 C CNN
 F 3 "" H 3300 2250 50  0001 C CNN
 	1    3300 2250
@@
 F 0 "R21" H 3425 3000 50  0000 C CNN
 F 1 "1k" H 3400 2900 50  0000 C CNN
-F 2 "Project:r-0805-hand-soldering" V 3230 2950 50  0001 C CNN
+F 2 "Project:r-1206-hand-soldering" V 3230 2950 50  0001 C CNN
 F 3 "" H 3300 2950 50  0001 C CNN
 	1    3300 2950
@@
 F 0 "R13" V 3150 1550 50  0000 C CNN
 F 1 "10K" V 3150 1375 50  0000 C CNN
-F 2 "Project:r-0805-hand-soldering" V 2980 1450 50  0001 C CNN
+F 2 "Project:r-1206-hand-soldering" V 2980 1450 50  0001 C CNN
 F 3 "" H 3050 1450 50  0001 C CNN
 	1    3050 1450
@@
 F 0 "R14" V 3150 3800 50  0000 C CNN
 F 1 "10K" V 3150 3625 50  0000 C CNN
-F 2 "Project:r-0805-hand-soldering" V 2980 3700 50  0001 C CNN
+F 2 "Project:r-1206-hand-soldering" V 2980 3700 50  0001 C CNN
 F 3 "" H 3050 3700 50  0001 C CNN
 	1    3050 3700
@@
 F 0 "R10" V 2625 1825 50  0000 C CNN
 F 1 "10K" V 2625 1650 50  0000 C CNN
-F 2 "Project:r-0805-hand-soldering" V 2480 1750 50  0001 C CNN
+F 2 "Project:r-1206-hand-soldering" V 2480 1750 50  0001 C CNN
 F 3 "" H 2550 1750 50  0001 C CNN
 	1    2550 1750
@@
 F 0 "R11" V 2625 2475 50  0000 C CNN
 F 1 "33K" V 2625 2275 50  0000 C CNN
-F 2 "Project:r-0805-hand-soldering" V 2480 2400 50  0001 C CNN
+F 2 "Project:r-1206-hand-soldering" V 2480 2400 50  0001 C CNN
 F 3 "" H 2550 2400 50  0001 C CNN
 	1    2550 2400
@@
 F 0 "R12" H 2675 3150 50  0000 C CNN
 F 1 "18K" H 2675 3050 50  0000 C CNN
-F 2 "Project:r-0805-hand-soldering" V 2730 3100 50  0001 C CNN
+F 2 "Project:r-1206-hand-soldering" V 2730 3100 50  0001 C CNN
 F 3 "" H 2800 3100 50  0001 C CNN
 	1    2800 3100
@@
 F 0 "R22" H 5675 1750 50  0000 C CNN
 F 1 "0R" H 5700 1650 50  0000 C CNN
-F 2 "Project:r-0805-hand-soldering" V 5730 1700 50  0001 C CNN
+F 2 "Project:r-1206-hand-soldering" V 5730 1700 50  0001 C CNN
 F 3 "" H 5800 1700 50  0001 C CNN
 	1    5800 1700
@@
 F 0 "R23" H 6125 1750 50  0000 C CNN
 F 1 "0R" H 6100 1650 50  0000 C CNN
-F 2 "Project:r-0805-hand-soldering" V 5930 1700 50  0001 C CNN
+F 2 "Project:r-1206-hand-soldering" V 5930 1700 50  0001 C CNN
 F 3 "" H 6000 1700 50  0001 C CNN
 	1    6000 1700
@@
 F 0 "R26" V 8130 4700 50  0000 C CNN
 F 1 "5K6" V 7950 4700 50  0000 C CNN
-F 2 "Project:r-0805-hand-soldering" V 7980 4700 50  0001 C CNN
+F 2 "Project:r-1206-hand-soldering" V 7980 4700 50  0001 C CNN
 F 3 "" H 8050 4700 50  0001 C CNN
 	1    8050 4700
@@
 F 0 "R30" V 8730 5400 50  0000 C CNN
 F 1 "10K" V 8550 5400 50  0000 C CNN
-F 2 "Project:r-0805-hand-soldering" V 8580 5400 50  0001 C CNN
+F 2 "Project:r-1206-hand-soldering" V 8580 5400 50  0001 C CNN
 F 3 "" H 8650 5400 50  0001 C CNN
 	1    8650 5400
@@
 F 0 "R24" V 7530 4000 50  0000 C CNN
 F 1 "5K6" V 7350 4000 50  0000 C CNN
-F 2 "Project:r-0805-hand-soldering" V 7380 4000 50  0001 C CNN
+F 2 "Project:r-1206-hand-soldering" V 7380 4000 50  0001 C CNN
 F 3 "" H 7450 4000 50  0001 C CNN
 	1    7450 4000
@@
 F 0 "R27" V 8230 4200 50  0000 C CNN
 F 1 "330K" V 8050 4200 50  0000 C CNN
-F 2 "Project:r-0805-hand-soldering" V 8080 4200 50  0001 C CNN
+F 2 "Project:r-1206-hand-soldering" V 8080 4200 50  0001 C CNN
 F 3 "" H 8150 4200 50  0001 C CNN
 	1    8150 4200
@@
 F 0 "R31" V 8830 4900 50  0000 C CNN
 F 1 "100K" V 8650 4900 50  0000 C CNN
-F 2 "Project:r-0805-hand-soldering" V 8680 4900 50  0001 C CNN
+F 2 "Project:r-1206-hand-soldering" V 8680 4900 50  0001 C CNN
 F 3 "" H 8750 4900 50  0001 C CNN
 	1    8750 4900
@@
 F 0 "R34" V 9480 5600 50  0000 C CNN
 F 1 "82K" V 9300 5600 50  0000 C CNN
-F 2 "Project:r-0805-hand-soldering" V 9330 5600 50  0001 C CNN
+F 2 "Project:r-1206-hand-soldering" V 9330 5600 50  0001 C CNN
 F 3 "" H 9400 5600 50  0001 C CNN
 	1    9400 5600
@@
 F 0 "R25" H 7550 5900 50  0000 C CNN
 F 1 "8K2" H 7550 5800 50  0000 C CNN
-F 2 "Project:r-0805-hand-soldering" V 7630 5850 50  0001 C CNN
+F 2 "Project:r-1206-hand-soldering" V 7630 5850 50  0001 C CNN
 F 3 "" H 7700 5850 50  0001 C CNN
 	1    7700 5850
@@
 F 0 "R28" H 8150 5900 50  0000 C CNN
 F 1 "3K9" H 8150 5800 50  0000 C CNN
-F 2 "Project:r-0805-hand-soldering" V 8230 5850 50  0001 C CNN
+F 2 "Project:r-1206-hand-soldering" V 8230 5850 50  0001 C CNN
 F 3 "" H 8300 5850 50  0001 C CNN
 	1    8300 5850
@@
 F 0 "R32" H 8750 5900 50  0000 C CNN
 F 1 "2K2" H 8750 5800 50  0000 C CNN
-F 2 "Project:r-0805-hand-soldering" V 8830 5850 50  0001 C CNN
+F 2 "Project:r-1206-hand-soldering" V 8830 5850 50  0001 C CNN
 F 3 "" H 8900 5850 50  0001 C CNN
 	1    8900 5850
@@
 F 0 "R29" H 8475 3100 50  0000 C CNN
 F 1 "880R" H 8450 3000 50  0000 C CNN
-F 2 "Project:r-0805-hand-soldering" V 8530 3050 50  0001 C CNN
+F 2 "Project:r-1206-hand-soldering" V 8530 3050 50  0001 C CNN
 F 3 "" H 8600 3050 50  0001 C CNN
 	1    8600 3050
@@
 F 0 "R33" H 9075 3100 50  0000 C CNN
 F 1 "220R" H 9050 3000 50  0000 C CNN
-F 2 "Project:r-0805-hand-soldering" V 9130 3050 50  0001 C CNN
+F 2 "Project:r-1206-hand-soldering" V 9130 3050 50  0001 C CNN
 F 3 "" H 9200 3050 50  0001 C CNN
 	1    9200 3050
@@
 F 0 "R35" H 9675 3100 50  0000 C CNN
 F 1 "1K2" H 9675 3000 50  0000 C CNN
-F 2 "Project:r-0805-hand-soldering" V 9730 3050 50  0001 C CNN
+F 2 "Project:r-1206-hand-soldering" V 9730 3050 50  0001 C CNN
 F 3 "" H 9800 3050 50  0001 C CNN
 	1    9800 3050
@@
 F 0 "R57" H 8875 1550 50  0000 C CNN
 F 1 "39K" H 8850 1450 50  0000 C CNN
-F 2 "Project:r-0805-hand-soldering" V 8930 1500 50  0001 C CNN
+F 2 "Project:r-1206-hand-soldering" V 8930 1500 50  0001 C CNN
 F 3 "" H 9000 1500 50  0001 C CNN
 	1    9000 1500
@@
 F 0 "R56" V 8880 1100 50  0000 C CNN
 F 1 "100R" V 8700 1100 50  0000 C CNN
-F 2 "Project:r-0805-hand-soldering" V 8730 1100 50  0001 C CNN
+F 2 "Project:r-1206-hand-soldering" V 8730 1100 50  0001 C CNN
 F 3 "" H 8800 1100 50  0001 C CNN
 	1    8800 1100

Commit message: Checks/Fixxes done, V1.0 ready for tape out
Parts:
- renumbered R57 to R49, R56 to R50
Changed lines of the file:
@@
 encoding utf-8
 Sheet 2 2
-Title ""
-Date ""
-Rev ""
-Comp ""
-Comment1 ""
+Title "RPI-EV-PLC Adapter"
+Date "2020-02-14"
+Rev "V1.0"
+Comp "(C) Manfred Steiner"
+Comment1 "https://github.com/greenenergyprojects/rpi-ev-plc-adapter"
 Comment2 ""
 Comment3 ""
@@
 $EndComp
 $Comp
-L Device:R R57
+L Device:R R49
 U 1 1 5E2785CA
 P 9000 1500
-F 0 "R57" H 8875 1550 50  0000 C CNN
+F 0 "R49" H 8875 1550 50  0000 C CNN
 F 1 "39K" H 8850 1450 50  0000 C CNN
 F 2 "Project:r-1206-hand-soldering" V 8930 1500 50  0001 C CNN
@@
 $EndComp
 $Comp
-L Device:R R56
+L Device:R R50
 U 1 1 5E29973A
 P 8800 1100
-F 0 "R56" V 8880 1100 50  0000 C CNN
+F 0 "R50" V 8880 1100 50  0000 C CNN
 F 1 "100R" V 8700 1100 50  0000 C CNN
 F 2 "Project:r-1206-hand-soldering" V 8730 1100 50  0001 C CNN

Commit message: Tapeout V1.0
Changed lines of the file:
@@
 AR Path="/5E34FA13" Ref="JP?"  Part="1"
 AR Path="/5E13857A/5E34FA13" Ref="JP3"  Part="1"
-F 0 "JP3" H 9750 1800 50  0000 L CNN
+F 0 "JP3" H 9725 1925 50  0000 L CNN
 F 1 "Jumper_NO_Small" V 9845 1898 50  0001 L CNN
 F 2 "Project:idc-header-1x02-p2.54mm-vertical" H 9800 1850 50  0001 C CNN
