File: kicad/rpi-ev-plc-adapter.kicad_pcb (KiCad board)
At the start: 4 copper layers, 65.1 x 56.6 mm, 103 parts, among them J1 Raspberry_RPI, J10 socket, J2 Conn_01x06, J3 header, J4 header, J5 header, J6 Screw_Terminal_01x04, J9 socket, M1 I2PLCAMN-ISE-002-T, M2 supply-5VtoPM12V_ebay-2530527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, Q1 AO3400, Q2 AO3401, Q3 AO3400, Q4 AO3401, SW1 push-button_ebay-183284526496, SW2 push-button_ebay-183284526496, SW3 SS-12D00G3, SW4 SS-12D00G3, SW5 dip-switch-6x2pos-smd-1.27mm, U1 LM224, U2 PC817C

Commit message: pcb fix for modem with 1.27mm connector finished
Parts:
- R37, R44: value 1G -> 3K3
- R38: value 47K -> 1G
- R7: value 47R -> 100R
- R9: value 22K -> 10K
- SW1, SW2: footprint Project:push-button_ebay-183284526496 -> Project:push-button-smd-4.5x4.5mm-black
- moved D8 11.7 mm to (-53.9, -14.1)
- moved D7 10.6 mm to (-49.0, -14.1)
- moved R44 10.4 mm to (-55.8, -5.42), turned to 90 degrees
- moved R42 7.78 mm to (-54.0, -5.42), turned to 90 degrees
- moved SW2 4.38 mm to (-49.4, -5.02)
- moved R45 4.28 mm to (-52.2, -5.42), turned to 90 degrees
- moved SW1 4.19 mm to (-49.4, -10.2)
- moved R43 2.34 mm to (-54.0, -10.1), turned to 90 degrees
- moved R23 2.29 mm to (-36.3, -18.9)
- moved R18 2.22 mm to (-41.3, -18.9)
- moved SW3 1.88 mm to (-42.0, -8.12)
- moved SW4 1.88 mm to (-36.8, -8.12)
- moved J2 0.28 mm to (-31.0, -16.0)
Connections:
- D8 pad 1: GND -> /CONNECTED
- M1 pad 15: /N -> Net-(M1-Pad15)
- M1 pad 18: (no net) -> Net-(M1-Pad18)
- M1 pad 25: (no net) -> Net-(M1-Pad25)
- R39 pad 2: /N -> Net-(M1-Pad15)
- R45 pad 1: /CONNECTED -> +3V3
Routing:
- net /Control-Pilot/VCPLT7V5: track 58.8 -> 30.3 mm, vias 2 -> 1
- net /N: track 42.1 -> 21.9 mm
- net /GPIO24: track 68.7 -> 84.2 mm, vias 1 -> 2
- net /GPIO25: track 68.7 -> 81.8 mm, vias 1 -> 2
- net Net-(R18-Pad1): track 12.6 -> 0.00 mm, vias 1 -> 0
- net /CONNECTED: track 58.7 -> 49.4 mm, vias 1 -> 0
- net Net-(C2-Pad1): track 64.6 -> 73.5 mm, vias 1 -> 3
- net +3V3: track 54.3 -> 63.1 mm, vias 14 -> 12
- net /PE: track 60.6 -> 54.3 mm
- net Net-(D1-Pad1): track 5.66 -> 0.00 mm
- net Net-(C3-Pad1): track 67.6 -> 72.9 mm, vias 1 -> 3
- net Net-(D8-Pad2): track 6.73 -> 11.3 mm
- net GND: track 81.5 -> 84.7 mm, vias 26 -> 24
- net Net-(M1-Pad15): track 0.00 -> 3.14 mm
- net /CONNECTING: track 65.3 -> 67.9 mm
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Other:
- board text added: "CON"
- board text added: "RES"
- board text added: "SCL"
- board text removed: "PLC CONNECT"
- board text removed: "PLC RESET"

Commit message: schematic/pcb V1.0 finished
Parts:
- removed R49, R50: 220R, Project:r-0805-hand-soldering
- C6: footprint Capacitors_THT:C_Disc_D3.8mm_W2.6mm_P2.50mm -> Project:c-1206-hand-soldering
- R1, R10, R11, R12, R13, R14, R15, R16, R17, R18, R19, R2, R20, R21, R22, R23, R24, R25, R26, R27, R28, R29, R3, R30, R31, R32, R33, R34, R35, R36, R37, R38, R39, R4, R40, R41, R42, R43, R44, R45, R46, R47, R5, R51, R52, R53, R54, R56, R57, R6, R7, R8, R9: footprint Project:r-0805-hand-soldering -> Project:r-1206-hand-soldering
- SW5: value dip-switch-6x2pos-smd-1.27mm -> dip-switch-4x2pos-smd-1.27mm; footprint Project:dip-switch-6x2pos-smd-1.27mm -> Project:dip-switch-4x2pos-smd-1.27mm
- moved R43 45.0 mm to (-9.56, -2.62), turned to 0 degrees
- moved D7 39.5 mm to (-10.9, -3.82)
- moved J4 16.0 mm to (6.64, -14.6), turned to 0 degrees
- moved R51 9.78 mm to (-0.46, -10.3), turned to 90 degrees
- moved D1 6.60 mm to (-45.9, -9.22), turned to 180 degrees
- moved Q3 6.00 mm to (-5.76, -5.22), turned to 270 degrees
- moved Q4 5.78 mm to (-13.9, -5.12), turned to 270 degrees
- moved R21 5.70 mm to (0.25, -17.2)
- moved R52 5.69 mm to (4.74, -3.02), turned to 0 degrees
- moved R10 5.61 mm to (-2.86, -6.12), turned to 90 degrees
- moved Q2 4.95 mm to (-5.76, -12.3), turned to 270 degrees
- moved R20 4.87 mm to (-2.76, -12.6), turned to 90 degrees
- moved C5 4.40 mm to (-41.9, -20.9), turned to 180 degrees
- moved R29 3.59 mm to (-32.3, -7.87), turned to 90 degrees
- moved R12 3.50 mm to (-11.0, -8.42), turned to 90 degrees
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Connections:
- net Net-(J1-Pad18) renamed /RECONN
- net Net-(M1-Pad3) renamed /SPIBURST
- J1 pad 13: Net-(J1-Pad13) -> (no net)
- J1 pad 15: Net-(J1-Pad15) -> (no net)
- J1 pad 22: Net-(J1-Pad22) -> /~PLC-RES
- J1 pad 26: Net-(J1-Pad26) -> /PI-IRQ
- J1 pad 32: Net-(J1-Pad32) -> /PI-PWM
- M1 pad 18: Net-(M1-Pad18) -> GND
- M1 pad 19: (no net) -> GND
- M1 pad 20: (no net) -> GND
- M1 pad 21: (no net) -> GND
- M1 pad 22: (no net) -> GND
- M1 pad 23: (no net) -> GND
- M1 pad 24: (no net) -> GND
- M1 pad 25: Net-(M1-Pad25) -> GND
- R2 pad 1: Net-(J1-Pad26) -> /PI-IRQ
- R36 pad 2: Net-(J1-Pad26) -> /PI-IRQ
- SW5 pad 1: Net-(J1-Pad32) -> /~PLC-RES
- SW5 pad 2: /PWM -> Net-(R3-Pad2)
- SW5 pad 4: Net-(R3-Pad2) -> Net-(R4-Pad2)
- SW5 pad 5: Net-(J1-Pad22) -> /PI-IRQ
- SW5 pad 6: Net-(R4-Pad2) -> /IRQ
- SW5 pad 7: Net-(J1-Pad26) -> /PI-PWM
- SW5 pad 8: /IRQ -> /PWM
Routing:
- net /CONNECTING: track 67.9 -> 126.8 mm, vias 2 -> 3
- net /PI-IRQ: track 0.00 -> 40.9 mm, vias 0 -> 1
- net /Control-Pilot/VCPLT7V5: track 30.3 -> 63.9 mm, vias 1 -> 4
- net /PI-PWM: track 0.00 -> 29.9 mm
- net Net-(J1-Pad32): track 23.2 -> 0.00 mm, vias 1 -> 0
- net Net-(R18-Pad1): track 0.00 -> 19.8 mm, vias 0 -> 1
- net GND: track 84.7 -> 104.2 mm
- net Net-(J1-Pad26): track 19.3 -> 0.00 mm, vias 2 -> 0
- net Net-(J1-Pad22): track 18.2 -> 0.00 mm
- net /PWM: track 66.1 -> 51.3 mm, vias 2 -> 1
- net /SCL1: track 10.3 -> 23.0 mm
- net /PE: track 54.3 -> 65.4 mm, vias 0 -> 2
- net Net-(D12-Pad2): track 15.5 -> 4.85 mm
- net Net-(J1-Pad13): track 9.85 -> 0.00 mm
- net /CONNECTED: track 49.4 -> 59.3 mm, vias 0 -> 1
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Other:
- board text added: "LCD-5V"
- board text removed: "(5V)"
- board text removed: "SMPL"

Commit message: Checks/Fixxes done, V1.0 ready for tape out
Parts:
- added J7: header, Project:idc-header-1x02-p2.54mm-vertical, F.Cu at (156.6, 96.8)
- added J8: header, Project:idc-header-1x02-p2.54mm-vertical, F.Cu at (156.7, 79.7)
- added R50: 100R, Project:r-0805-hand-soldering, B.Cu at (155.0, 73.7)
- R56: value 100R -> 0R
- moved C8 181.3 mm to (157.0, 72.4)
- moved R49 180.8 mm to (154.4, 79.7)
- moved C1 180.3 mm to (109.8, 58.8)
- moved C2 180.3 mm to (123.2, 54.7)
- moved C3 180.3 mm to (132.9, 63.2)
- moved C4 180.3 mm to (109.0, 63.5)
- moved C5 180.3 mm to (108.1, 79.1)
- moved D1 180.3 mm to (104.1, 90.8)
- moved D10 180.3 mm to (134.6, 51.8)
- moved D11 180.3 mm to (128.8, 51.8)
- moved D12 180.3 mm to (150.0, 96.2)
- moved D13 180.3 mm to (146.8, 57.7)
- moved D2 180.3 mm to (110.0, 76.6)
- moved D3 180.3 mm to (99.9, 74.3)
- moved D4 180.3 mm to (119.1, 89.3)
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- renumbered R57 to R49
Connections:
- R56 pad 1: +3V3 -> GND
- R56 pad 2: Net-(C8-Pad1) -> /PE
Routing:
- net GND: track 104.2 -> 124.3 mm, vias 24 -> 23
- net /SDA1: track 15.9 -> 32.7 mm
- net /PE: track 65.4 -> 68.7 mm
- net +3V3: track 61.9 -> 58.6 mm, vias 14 -> 15
- net +5V: track 31.1 -> 34.1 mm
- net Net-(D7-Pad2): track 6.41 -> 8.43 mm
- net /SCL1: track 23.0 -> 21.7 mm
- net Net-(C8-Pad1): track 5.29 -> 6.54 mm
- net /5V-LCD: track 10.1 -> 9.28 mm
- net /Control-Pilot/L: track 3.68 -> 3.06 mm
Other:
- board text added: "+12V"
- board text added: "+3.3V"
- board text added: "+5V"
- board text added: "-12V"

Commit message: Tapeout V1.0
Parts:
- added R57: 10G, Project:r-0805-hand-soldering, B.Cu at (94.4, 88.8)
- R36, R38, R42: value 1G -> 10G; footprint Project:r-1206-hand-soldering -> Project:r-0805-hand-soldering
- R40, R41: value 1G -> 0R
- R50: footprint Project:r-0805-hand-soldering -> Project:r-1206-hand-soldering
- R53, R54: value 0R -> 10G; footprint Project:r-1206-hand-soldering -> Project:r-0805-hand-soldering
- moved R56 26.8 mm to (131.9, 81.2), turned to 0 degrees
- moved D12 3.19 mm to (146.8, 96.2)
- moved C8 2.13 mm to (154.9, 72.8)
- moved R50 2.13 mm to (156.9, 72.7), turned to 90 degrees
- moved D7 1.96 mm to (137.2, 96.2)
- moved R36 1.62 mm to (126.4, 93.2)
- moved R5 1.23 mm to (125.4, 81.2)
- moved R38 0.71 mm to (96.1, 61.7)
- moved R53 0.68 mm to (128.1, 74.0)
- moved R54 0.68 mm to (135.0, 74.0)
- moved R44 0.38 mm to (94.4, 94.4)
Routing:
- net GND: track 124.3 -> 130.2 mm, vias 23 -> 24
- net Net-(D12-Pad2): track 4.85 -> 7.62 mm
- net /PWM: track 51.4 -> 53.4 mm, vias 1 -> 2
- net Net-(C8-Pad1): track 6.54 -> 8.46 mm
- net Net-(D8-Pad2): track 10.7 -> 9.18 mm
- net /SCL1: track 21.7 -> 23.0 mm
- net /PI-IRQ: track 40.9 -> 42.2 mm
- net /SDA1: track 32.7 -> 33.8 mm
- net /PE: track 68.7 -> 69.8 mm
- net /Control-Pilot/VCPLT3V5: track 48.5 -> 47.9 mm
- net /MISO: track 65.4 -> 64.8 mm
- net Net-(R3-Pad2): track 33.9 -> 33.3 mm
- net /SCLK: track 68.0 -> 67.4 mm
- net Net-(R4-Pad2): track 28.5 -> 29.0 mm
- net /CONNECTING: track 126.6 -> 126.1 mm
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Other:
- board text added: "3.3V"
