File: kicad/rpi-ev-plc-adapter.sch (KiCad schematic (older format))
At the start: 51 parts, among them J1 Raspberry_RPI, J10 socket, J2 Conn_01x06, J3 header, J4 header, J5 header, J7 header, J8 header, J9 socket, M1 I2PLCAMN-ISE-002-T, M2 supply-5VtoPM12V_ebay-2530527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, SW1 push-button_ebay-183284526496, SW2 push-button_ebay-183284526496, SW5 dip-switch-4x2pos-smd-1.27mm

Commit message: Tapeout V1.0
Parts:
- added R56: 0R, Project:r-1206-hand-soldering, symbol Device:R
- added R57: 10G, Project:r-0805-hand-soldering, symbol Device:R
- R36, R38, R42: value 1G -> 10G; footprint Project:r-1206-hand-soldering -> Project:r-0805-hand-soldering
- R40, R41: value 1G -> 0R
- R53, R54: value 0R -> 10G; footprint Project:r-1206-hand-soldering -> Project:r-0805-hand-soldering
Connections:
- net CONNECTED: now also R57.1
- net GND: now also R56.1, R57.2
- net PE: now also R56.2
Changed lines of the file:
@@
 P 6100 4500
 F 0 "R36" H 5900 4600 50  0000 L CNN
-F 1 "1G" H 5900 4500 50  0000 L CNN
-F 2 "Project:r-1206-hand-soldering" V 6030 4500 50  0001 C CNN
+F 1 "10G" H 5900 4500 50  0000 L CNN
+F 2 "Project:r-0805-hand-soldering" V 6030 4500 50  0001 C CNN
 F 3 "~" H 6100 4500 50  0001 C CNN
 	1    6100 4500
@@
 P 7600 2450
 F 0 "R38" H 7650 2450 50  0000 L CNN
-F 1 "1G" H 7400 2450 50  0000 L CNN
-F 2 "Project:r-1206-hand-soldering" V 7530 2450 50  0001 C CNN
+F 1 "10G" H 7400 2450 50  0000 L CNN
+F 2 "Project:r-0805-hand-soldering" V 7530 2450 50  0001 C CNN
 F 3 "~" H 7600 2450 50  0001 C CNN
 	1    7600 2450
@@
 P 10175 4850
 F 0 "R42" H 9975 4900 50  0000 L CNN
-F 1 "1G" H 10025 4800 50  0000 L CNN
-F 2 "Project:r-1206-hand-soldering" V 10105 4850 50  0001 C CNN
+F 1 "10G" H 9975 4800 50  0000 L CNN
+F 2 "Project:r-0805-hand-soldering" V 10105 4850 50  0001 C CNN
 F 3 "~" H 10175 4850 50  0001 C CNN
 	1    10175 4850
@@
 P 9650 3550
 F 0 "R40" H 9450 3600 50  0000 L CNN
-F 1 "1G" H 9500 3500 50  0000 L CNN
+F 1 "0R" H 9500 3500 50  0000 L CNN
 F 2 "Project:r-1206-hand-soldering" V 9580 3550 50  0001 C CNN
 F 3 "~" H 9650 3550 50  0001 C CNN
@@
 P 9850 3550
 F 0 "R41" H 9900 3600 50  0000 L CNN
-F 1 "1G" H 9900 3500 50  0000 L CNN
+F 1 "0R" H 9900 3500 50  0000 L CNN
 F 2 "Project:r-1206-hand-soldering" V 9780 3550 50  0001 C CNN
 F 3 "~" H 9850 3550 50  0001 C CNN
@@
 	1900 2700 1400 2700
 Wire Wire Line
-	1400 2700 1400 1350
+	1400 2700 1400 2200
 Connection ~ 1400 1350
 Wire Wire Line
@@
 P 10300 3550
 F 0 "R53" H 10100 3600 50  0000 L CNN
-F 1 "0R" H 10125 3500 50  0000 L CNN
-F 2 "Project:r-1206-hand-soldering" V 10230 3550 50  0001 C CNN
+F 1 "10G" H 10100 3500 50  0000 L CNN
+F 2 "Project:r-0805-hand-soldering" V 10230 3550 50  0001 C CNN
 F 3 "~" H 10300 3550 50  0001 C CNN
 	1    10300 3550
@@
 P 10500 3550
 F 0 "R54" H 10550 3600 50  0000 L CNN
-F 1 "0R" H 10550 3500 50  0000 L CNN
-F 2 "Project:r-1206-hand-soldering" V 10430 3550 50  0001 C CNN
+F 1 "10G" H 10550 3500 50  0000 L CNN
+F 2 "Project:r-0805-hand-soldering" V 10430 3550 50  0001 C CNN
 F 3 "~" H 10500 3550 50  0001 C CNN
 	1    10500 3550
@@
 Wire Wire Line
 	4550 1200 4600 1200
+$Comp
+L Device:R R56
+U 1 1 5E597788
+P 1100 2200
+F 0 "R56" V 1000 2300 50  0000 C CNN
+F 1 "0R" V 1000 2100 50  0000 C CNN
+F 2 "Project:r-1206-hand-soldering" V 1030 2200 50  0001 C CNN
+F 3 "~" H 1100 2200 50  0001 C CNN
+	1    1100 2200
+	0    -1   1    0
+$EndComp
+Wire Wire Line
+	1400 2200 1250 2200
+Connection ~ 1400 2200
+Wire Wire Line
+	1400 2200 1400 1350
+$Comp
+L power:GND #PWR0146
+U 1 1 5E5A9F92
+P 875 2300
+F 0 "#PWR0146" H 875 2050 50  0001 C CNN
+F 1 "GND" H 880 2127 50  0000 C CNN
+F 2 "" H 875 2300 50  0001 C CNN
+F 3 "" H 875 2300 50  0001 C CNN
+	1    875  2300
+	1    0    0    -1
+$EndComp
+Wire Wire Line
+	950  2200 875  2200
+Wire Wire Line
+	875  2200 875  2300
+$Comp
+L Device:R R57
+U 1 1 5E49A704
+P 10800 5400
+F 0 "R57" H 10600 5450 50  0000 L CNN
+F 1 "10G" H 10575 5350 50  0000 L CNN
+F 2 "Project:r-0805-hand-soldering" V 10730 5400 50  0001 C CNN
+F 3 "~" H 10800 5400 50  0001 C CNN
+	1    10800 5400
+	1    0    0    -1
+$EndComp
+$Comp
+L power:GND #PWR0159
+U 1 1 5E49A7DA
+P 10800 5650
+F 0 "#PWR0159" H 10800 5400 50  0001 C CNN
+F 1 "GND" H 10805 5477 50  0000 C CNN
+F 2 "" H 10800 5650 50  0001 C CNN
+F 3 "" H 10800 5650 50  0001 C CNN
+	1    10800 5650
+	1    0    0    -1
+$EndComp
+Wire Wire Line
+	10800 5100 10800 5250
+Connection ~ 10800 5100
+Wire Wire Line
+	10800 5550 10800 5650
 $EndSCHEMATC
