File: kicad-backup/control-pilot.sch (KiCad schematic (older format))
At the start: 52 parts, among them J6 Screw_Terminal_01x04, Q1 AO3400, Q2 AO3401, Q3 AO3400, Q4 AO3401, SW3 SS-12D00G3, SW4 SS-12D00G3, U1 LM224, U2 PC817C

Commit message: removing rescue lib
Parts:
- C5: symbol Device:C -> rpi-ev-plc-adapter-rescue:C-ev-charger-met16-rescue
- D1, D2: symbol project:B5819WS -> rpi-ev-plc-adapter-rescue:D_Schottky-ev-charger-met16-rescue
- R10, R11, R12, R13, R14, R15, R16, R17, R18, R19, R20, R21, R22, R23, R24, R25, R26, R27, R28, R29, R30, R31, R32, R33, R34, R35, R55, R56, R57: symbol Device:R -> rpi-ev-plc-adapter-rescue:R-ev-charger-met16-rescue
Changed lines of the file:
@@
 $EndDescr
 $Comp
-L Device:R R15
+L rpi-ev-plc-adapter-rescue:R-ev-charger-met16-rescue R15
 U 1 1 5AB4B011
 P 4500 3450
@@
 $EndComp
 $Comp
-L Device:R R16
+L rpi-ev-plc-adapter-rescue:R-ev-charger-met16-rescue R16
 U 1 1 5AB4B086
 P 4500 4050
@@
 $EndComp
 $Comp
-L Device:C C5
+L rpi-ev-plc-adapter-rescue:C-ev-charger-met16-rescue C5
 U 1 1 5AB4B858
 P 6000 4050
@@
 $EndComp
 $Comp
-L project:B5819WS D2
+L rpi-ev-plc-adapter-rescue:D_Schottky-ev-charger-met16-rescue D2
 U 1 1 5AB4A9B7
 P 5600 3800
@@
 $EndComp
 $Comp
-L Device:R R19
+L rpi-ev-plc-adapter-rescue:R-ev-charger-met16-rescue R19
 U 1 1 5AB4C124
 P 6300 4050
@@
 Simulate car
 $Comp
-L Device:R R17
+L rpi-ev-plc-adapter-rescue:R-ev-charger-met16-rescue R17
 U 1 1 5AE42C8F
 P 5800 1300
@@
 $EndComp
 $Comp
-L Device:R R18
+L rpi-ev-plc-adapter-rescue:R-ev-charger-met16-rescue R18
 U 1 1 5AE42DED
 P 6000 1300
@@
 $EndComp
 $Comp
-L project:B5819WS D1
+L rpi-ev-plc-adapter-rescue:D_Schottky-ev-charger-met16-rescue D1
 U 1 1 5AE44F46
 P 4650 1000
@@
 $EndComp
 $Comp
-L Device:R R20
+L rpi-ev-plc-adapter-rescue:R-ev-charger-met16-rescue R20
 U 1 1 5E207D03
 P 3300 2250
@@
 $EndComp
 $Comp
-L Device:R R21
+L rpi-ev-plc-adapter-rescue:R-ev-charger-met16-rescue R21
 U 1 1 5E207ED7
 P 3300 2950
@@
 $EndComp
 $Comp
-L Device:R R13
+L rpi-ev-plc-adapter-rescue:R-ev-charger-met16-rescue R13
 U 1 1 5E208145
 P 3050 1450
@@
 $EndComp
 $Comp
-L Device:R R14
+L rpi-ev-plc-adapter-rescue:R-ev-charger-met16-rescue R14
 U 1 1 5E20831F
 P 3050 3700
@@
 $EndComp
 $Comp
-L Device:R R10
+L rpi-ev-plc-adapter-rescue:R-ev-charger-met16-rescue R10
 U 1 1 5E2168AF
 P 2550 1750
@@
 	2800 2950 2800 2900
 $Comp
-L Device:R R11
+L rpi-ev-plc-adapter-rescue:R-ev-charger-met16-rescue R11
 U 1 1 5E229C3D
 P 2550 2400
@@
 	1600 2050 1700 2050
 $Comp
-L Device:R R12
+L rpi-ev-plc-adapter-rescue:R-ev-charger-met16-rescue R12
 U 1 1 5E2522B7
 P 2800 3100
@@
 CP
 $Comp
-L Device:R R22
+L rpi-ev-plc-adapter-rescue:R-ev-charger-met16-rescue R22
 U 1 1 5E29E1DE
 P 5800 1700
@@
 $EndComp
 $Comp
-L Device:R R23
+L rpi-ev-plc-adapter-rescue:R-ev-charger-met16-rescue R23
 U 1 1 5E29E22A
 P 6000 1700
@@
 	7000 3800 7000 4500
 $Comp
-L Device:R R26
+L rpi-ev-plc-adapter-rescue:R-ev-charger-met16-rescue R26
 U 1 1 5E104ECB
 P 8050 4700
@@
 $EndComp
 $Comp
-L Device:R R30
+L rpi-ev-plc-adapter-rescue:R-ev-charger-met16-rescue R30
 U 1 1 5E105011
 P 8650 5400
@@
 $EndComp
 $Comp
-L Device:R R24
+L rpi-ev-plc-adapter-rescue:R-ev-charger-met16-rescue R24
 U 1 1 5E1050C0
 P 7450 4000
@@
 $EndComp
 $Comp
-L Device:R R27
+L rpi-ev-plc-adapter-rescue:R-ev-charger-met16-rescue R27
 U 1 1 5E10A656
 P 8150 4200
@@
 $EndComp
 $Comp
-L Device:R R31
+L rpi-ev-plc-adapter-rescue:R-ev-charger-met16-rescue R31
 U 1 1 5E10A6E2
 P 8750 4900
@@
 $EndComp
 $Comp
-L Device:R R34
+L rpi-ev-plc-adapter-rescue:R-ev-charger-met16-rescue R34
 U 1 1 5E10A78A
 P 9400 5600
@@
 $EndComp
 $Comp
-L Device:R R25
+L rpi-ev-plc-adapter-rescue:R-ev-charger-met16-rescue R25
 U 1 1 5E10FD6C
 P 7700 5850
@@
 $EndComp
 $Comp
-L Device:R R28
+L rpi-ev-plc-adapter-rescue:R-ev-charger-met16-rescue R28
 U 1 1 5E10FE52
 P 8300 5850
@@
 $EndComp
 $Comp
-L Device:R R32
+L rpi-ev-plc-adapter-rescue:R-ev-charger-met16-rescue R32
 U 1 1 5E10FF0C
 P 8900 5850
@@
 	8900 5600 8900 5400
 $Comp
-L Device:R R29
+L rpi-ev-plc-adapter-rescue:R-ev-charger-met16-rescue R29
 U 1 1 5E15A44D
 P 8600 3050
@@
 	8600 2900 8600 2800
 $Comp
-L Device:R R33
+L rpi-ev-plc-adapter-rescue:R-ev-charger-met16-rescue R33
 U 1 1 5E16B5C8
 P 9200 3050
@@
 	9200 2900 9200 2800
 $Comp
-L Device:R R35
+L rpi-ev-plc-adapter-rescue:R-ev-charger-met16-rescue R35
 U 1 1 5E16FA1F
 P 9800 3050
@@
 	6000 2200 5800 2200
 $Comp
-L Device:R R55
+L rpi-ev-plc-adapter-rescue:R-ev-charger-met16-rescue R55
 U 1 1 5E245DB5
 P 7700 1400
@@
 $EndComp
 $Comp
-L Device:R R57
+L rpi-ev-plc-adapter-rescue:R-ev-charger-met16-rescue R57
 U 1 1 5E2785CA
 P 9000 1500
@@
 $EndComp
 $Comp
-L Device:R R56
+L rpi-ev-plc-adapter-rescue:R-ev-charger-met16-rescue R56
 U 1 1 5E29973A
 P 8800 1100
