File: kicad-backup/rpi-ev-plc-adapter.sch (KiCad schematic (older format))
At the start: 51 parts, among them J1 Raspberry_RPI, J10 socket, J2 Conn_01x06, J3 header, J4 header, J5 header, J9 socket, M1 I2PLCAMN-ISE-002-T, M2 supply-5VtoPM12V_ebay-2530527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, SW1 push-button_ebay-183284526496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

Commit message: removing rescue lib
Parts:
- R43, R45, R46, R47, R48: symbol Device:R -> rpi-ev-plc-adapter-rescue:R-ev-charger-met16-rescue
Changed lines of the file:
@@
 L-B
 $Comp
-L Device:R R?
+L rpi-ev-plc-adapter-rescue:R-ev-charger-met16-rescue R?
 U 1 1 5E2A00E2
 P 10750 5550
@@
 	10750 6100 10750 6200
 $Comp
-L Device:R R?
+L rpi-ev-plc-adapter-rescue:R-ev-charger-met16-rescue R?
 U 1 1 5E2C2D62
 P 10300 5550
@@
 	3250 2500 3350 2500
 $Comp
-L Device:R R?
+L rpi-ev-plc-adapter-rescue:R-ev-charger-met16-rescue R?
 U 1 1 5E85A611
 P 2500 5350
@@
 	2500 5200 2500 4800
 $Comp
-L Device:R R?
+L rpi-ev-plc-adapter-rescue:R-ev-charger-met16-rescue R?
 U 1 1 5E866216
 P 2900 5350
@@
 	2900 5200 2900 4900
 $Comp
-L Device:R R?
+L rpi-ev-plc-adapter-rescue:R-ev-charger-met16-rescue R?
 U 1 1 5E8724DA
 P 3300 5350
